File: dcdc 1.1 0223.sch (EAGLE design)
At the start: 21 parts, among them M1 BSS97, X2 OUTPUT

Commit message: second commit
Parts:
- removed PIN: Input, con-garry:332-06
- removed X2: OUTPUT, con-garry:332-02
- added C4: (no value), rcl:C-US050-050X075
- added IN, OUT: XT30UPB-M, amass:XT30UPB-M
- added JP1: PINHD-1X2, Connector:PINHD-1X2
- renumbered CIN to C9, COUT to C8, CPRI1 to C1, CPRI2 to C2, CPRI3 to C3, FWFD to C7
Connections:
- net 66 renamed SOURCE
- removed net N$15: PIN-5.S, R7.1, U$1.P$3
- removed net N$9: DOUT.A, U$2.P$3
- new net N$5: JP1.1, R7.1, U$1.P$3
- new net N$7: DOUT.A, U$2.P$1
- net 0: now also C4.2, IN.-, OUT.-, U$2.P$6; no longer PIN-4.S, U$2.P$4, X2-2.S
- net DRAIN: now also U$2.P$10, U$2.P$9; no longer U$2.P$2
- net N$10: now also OUT.+; no longer X2-1.S
- net N$13: now also C4.1, IN.+, U$2.P$4, U$2.P$5; no longer PIN-6.S, U$2.P$1
- net N$8: now also JP1.2; no longer PIN-2.S
